File: reader_shield/flash.kicad_sch (KiCad schematic)
At the start: 1 part, among them U1 MX29GL128FHT2I-90G

Commit message: Describe sheets
Other:
- company: (none) -> rwilliaise
- title: (none) -> reader00 Shield Flash
Changed lines of the file:
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@@
 (kicad_sch (version 20230121) (generator eeschema)
-  (paper "A4")
+  (paper "USLetter")
+  (title_block
+    (title "reader00 Shield Flash")
+    (rev "1")
+    (company "rwilliaise")
+  )
   (junction (at 137.16 129.54) (diameter 0) (color 0 0 0 0)
   )

Commit message: Revisions 1 and 2
Parts:
- added C13, C4: 0.1u, Capacitor_SMD:C_0402_1005Metric, symbol Device:C_Small
- added D1: 520, LED_SMD:LED_0603_1608Metric, symbol Device:LED_Small
- added R1: 200, Resistor_SMD:R_0603_1608Metric, symbol Device:R_Small
Connections:
- net +3V3: now also U1.13 (WE), U1.14 (RESET), U1.29 (VI/0), U1.53 (BYTE), C13.2, C4.2, R1.2
- net GND: now also C13.1, C4.1
- net at U1.17 (RY): now also D1.1 (K)
- net D9: now reaches U1.32 (CE)
- net D10: now reaches U1.34 (OE)
- new net: D1.2 (A), R1.1
